File: schematic/LiFePO4-Charge-Controller.sch (KiCad schematic (older format))
At the start: 47 parts, among them IC1 PC817, IC2 PC817, IC3 PC817, P1 CONN_2, P2 CONN_4, P3 CONN_4, P4 CONN_4, P5 CONN_4, P6 CONN_4, P7 CONN_2, P8 CONN_2, P9 CONN_2, Q1 NPN, U1 AD8236, U2 SI8400, U3 SI8400, U4 ARDUINO_MINI, U5 SI8400

Commit message: Autoraouted board b4 contraction
Parts:
- added Dled1, Dled2: LED, ~, symbol LED
- added Rled1: 1k, ~, symbol R
- added Rled2: 1K, ~, symbol R
- CI1a1: renamed from C8; value C -> 100nF
- CI1b1: renamed from C9; value C -> 1uF
- CI1c1: renamed from C1; value C -> 100nF
- CI1d1: renamed from C2; value C -> 1uF
- CI2a1: renamed from C6; value C -> 100nF
- CI2b1: renamed from C7; value C -> 1uF
- CI2c1: renamed from C3; value C -> 100nF
- CI2d1: renamed from C4; value C -> 1uF
- CI3a1: renamed from C10; value C -> 100nF
- CI3b1: renamed from C11; value C -> 1uF
- CINA1: renamed from C5; value C -> 100nF
- CV1: renamed from C13; value C -> 10pF
- Cpwm1: renamed from C12; value C -> 300nF
- PI1: renamed from P2; value CONN_4 -> I2C
- PI2: renamed from P3; value CONN_4 -> I2C
- PI2C1: renamed from P6; value CONN_4 -> I2C
- PIRS232: renamed from P5; value CONN_4 -> RS232
- Popto1: renamed from P7; value CONN_2 -> opto
- Popto2: renamed from P8; value CONN_2 -> opto
- Popto3: renamed from P9; value CONN_2 -> opto
- Pshunt1: renamed from P1; value CONN_2 -> differential
- Pvolt1: renamed from P4; value CONN_4 -> Gnd PWM 12V B+
- RI1scl1: renamed from R2; value R -> 5k
- RI1sda1: renamed from R4; value R -> 5k
- RI2Cscl1: renamed from R6; value R -> 1.8k
- RI2Csda1: renamed from R5; value R -> 1.8k
- RI2scl1: renamed from R1; value R -> 5k
- RI2sda1: renamed from R3; value R -> 5k
- Rg1: renamed from RV1; value POT -> 5k
- Ropto1: renamed from R13; value R -> 1k
- Ropto2: renamed from R14; value R -> 1k
- Ropto3: renamed from R15; value R -> 1k
- Rpwm1: renamed from R7; value R -> 120
- UuC1: renamed from U4; value ARDUINO_MINI -> ARDUINO_Nano
- renumbered IC1 to OC1, IC2 to OC2, IC3 to OC3, Q1 to Qpnp1, R8 to RVR1a1, R10 to RVR1b1, R9 to RVR2a1, R11 to RVR2b1, R12 to RpwmDrv1, U2 to UI1, U3 to UI2, U1 to UINA1, U5 to UIR1
Connections:
- wire segments 143 -> 148

Commit message: PCB satisfactory, bit of a mess around I2C, but will go with it
Connections:
- net labels added: I2C1_GND, I2C2_GND, RS232_GND
- wire segments 148 -> 149
Changed lines of the file:
@@
 	1500 5350 1400 5350
 Wire Wire Line
-	1400 5550 1500 5550
+	1300 5550 1500 5550
 Wire Wire Line
 	2050 4100 1900 4100
@@
 	1500 3900 1400 3900
 Wire Wire Line
-	1400 4100 1500 4100
+	1300 4100 1500 4100
 Wire Wire Line
 	1300 5200 2100 5200
@@
 Connection ~ 7650 3550
 Connection ~ 7650 2900
+Connection ~ 1400 4100
+Connection ~ 1400 5550
+Wire Wire Line
+	8850 4250 8850 4400
+Text GLabel 1300 4100 0    60   Input ~ 0
+I2C1_GND
+Text GLabel 1300 5550 0    60   Input ~ 0
+I2C2_GND
+Text GLabel 8850 4400 3    60   Input ~ 0
+RS232_GND
 $EndSCHEMATC

Commit message: PWM/PID code corrected. PCB: In-Amp pad (module) corrected. Board done.
Changed lines of the file:
@@
 Sheet 1 1
 Title ""
-Date "29 jul 2014"
+Date "30 jul 2014"
 Rev ""
 Comp ""
@@
 Text GLabel 8850 4400 3    60   Input ~ 0
 RS232_GND
+Connection ~ 4000 1550
 $EndSCHEMATC

Commit message: moving to another computer. PCB: Moving to new version of Kicad, and making resistors SMD etc
Parts:
- added D1: DIODESCH, ~, symbol DIODESCH
Connections:
- wire segments 149 -> 151
Changed lines of the file:
@@
 Sheet 1 1
 Title ""
-Date "30 jul 2014"
+Date "9 aug 2014"
 Rev ""
 Comp ""
@@
 RS232_GND
 Connection ~ 4000 1550
+$Comp
+L DIODESCH D1
+U 1 1 53E68BE4
+P 4750 2450
+F 0 "D1" H 4750 2550 40  0000 C CNN
+F 1 "DIODESCH" H 4750 2350 40  0000 C CNN
+F 2 "~" H 4750 2450 60  0000 C CNN
+F 3 "~" H 4750 2450 60  0000 C CNN
+	1    4750 2450
+	-1   0    0    1
+$EndComp
+Wire Wire Line
+	4950 2450 5000 2450
+Connection ~ 5000 2450
+Wire Wire Line
+	4550 2450 4500 2450
+Connection ~ 4500 2450
 $EndSCHEMATC

Commit message: Modified schematic to incorporate fix on PWM output, still working on non tracked test code
Parts:
- removed UI1, UI2, UIR1: SI8400, MODULE, symbol SI8400
- removed UuC1: ARDUINO_Nano, DIL20, symbol ARDUINO_MINI
- added U1, UI1, UI2: Si8400, SO8E, symbol Si8400
- added UcC1: arduino_mini, arduino_mini, symbol arduino_mini
- Cpwm1: value 300nF -> 1uF
- Qpnp1: footprint ~ -> SOT-23-EBC
- RVR1a1, RVR1b1: value 99k -> 47k
- RVR2a1, RVR2b1: value 1k -> 4k7
- Rpwm1: value 120 -> 100
Other:
- moved on the sheet: OC1, OC2, OC3, Popto1, Popto2, Popto3, Qpnp1, Ropto1, Ropto2, Ropto3, Rpwm1

Commit message: Basic working solution
Parts:
- added Rpwm2: 1k, symbol R
- added UPWM: LMC662, symbol TL071
- Cpwm1: value 1uF -> 10u
- RVR1a1, RVR1b1: value 47k -> 470k
- Rpwm1: value 100 -> 1K
Connections:
- wire segments 151 -> 159
Other:
- moved on the sheet: CV1, Cpwm1, Pvolt1, Qpnp1, RVR1a1, RVR1b1, RVR2a1, RVR2b1, Rpwm1
